Commit message: Add web teleop and slam_toolbox bringup.
This adds an agv_bringup web teleop (8080) with rosbridge (9090) and introduces a slam_toolbox-based bringup launch with optional RViz and TF support.

Made-with: Cursor

File: src/agv_description/urdf/b300_description.urdf.xacro (robot description, xacro)
@@ -6,6 +6,6 @@
   <xacro:property name="lidar_cylinder_length" value="0.03" />
   <xacro:property name="lidar_mount_z" value="0.185" />
-  <xacro:property name="imu_mount_x"   value="-0.225" />
-  <xacro:property name="imu_mount_y"   value="-0.135" />
+  <xacro:property name="imu_mount_x"   value="0" />
+  <xacro:property name="imu_mount_y"   value="0" />
   <xacro:property name="imu_mount_z"   value="0.0" />
   <xacro:property name="imu_mount_rpy" value="0 0 0" />
